File: Safesteps.kicad_sch (KiCad schematic)
At the start: 12 parts, among them J1 Conn_01x06_Pin, J2 Conn_01x05_Pin, SW1 SW_Push, U3 3.3 V, U4 ESP32-DEVKIT-V1

Commit message: Page Settings
Other:
- note added: "SafeSteps"
- note removed: "Neo-6M GPS"
- company: (none) -> Final year project 
- title: (none) -> Safesteps women safety device 
- moved on the sheet: AE1, BT1, BZ1, C1, C2, D1, J1, J2, R1, SW1, U3, U4

Commit message: Layout design Settings
Parts:
- added H1, H2, H3, H4: MountingHole, MountingHole:MountingHole_2.1mm, symbol Mechanical:MountingHole
- SW1: footprint Button_Switch_THT:SW_NKK_GW12LJP -> Button_Switch_THT:SW_PUSH-12mm
Other:
- note added: "Mouting holes"
